Commit message: add files for peng

File: gazebo_ros_demos/rrbot_description/urdf/rrbot.xacro (robot description, xacro)
@@ -50,5 +50,5 @@
     <origin xyz="0 ${width} ${height1 - axel_offset}" rpy="0 0 0"/>
     <axis xyz="0 1 0"/>
-    <limit effort="10" lower="${-PI*2.0}" upper="${PI*2.0}" velocity="1"/>
+    <limit effort="1000" lower="${-PI*2.0}" upper="${PI*2.0}" velocity="1"/>
     <dynamics damping="0.1"/>
   </joint>
@@ -82,5 +82,5 @@
     <origin xyz="0 ${width} ${height2 - axel_offset*2}" rpy="0 0 0"/>
     <axis xyz="0 1 0"/>
-    <limit effort="10" lower="${-PI*2.0}" upper="${PI*2.0}" velocity="1"/>
+    <limit effort="1000" lower="${-PI*2.0}" upper="${PI*2.0}" velocity="1"/>
     <dynamics damping="0.1"/>
   </joint>
