Commit message: change peng's script

File: gazebo_ros_demos/rrbot_description/urdf/rrbot_two.xacro (robot description, xacro)
@@ -233,8 +233,8 @@
     <inertial>
       <origin xyz="0 0.0 0" rpy="0 0 0"/>
-      <mass value="0.001"/>
-      <inertia
-	  ixx="1" ixy="0.0" ixz="0.0"
-	  iyy="1" iyz="0.0"
+      <mass value="10"/>
+      <inertia
+	  ixx="10" ixy="0.0" ixz="0.0"
+	  iyy="10" iyz="0.0"
 	  izz="0"/>
     </inertial>
@@ -244,15 +244,12 @@
     <child link="box"/>
     <origin xyz="0 ${width} ${height3 - axel_offset*2}" rpy="0 0 0"/>
-    <!-- <axis xyz="0 1 0"/> -->
-    <!-- <limit effort="1000" lower="${-PI*2.0}" upper="${PI*2.0}" velocity="1"/> -->
-    <!-- <dynamics damping="0.1"/> -->
   </joint>
   <link name="box_copy">
     <inertial>
       <origin xyz="0 0.0 0" rpy="0 0 0"/>
-      <mass value="0.001"/>
-      <inertia
-	  ixx="1" ixy="0.0" ixz="0.0"
-	  iyy="1" iyz="0.0"
+      <mass value="10"/>
+      <inertia
+	  ixx="10" ixy="0.0" ixz="0.0"
+	  iyy="10" iyz="0.0"
 	  izz="0"/>
     </inertial>

Commit message: wtf

File: gazebo_ros_demos/rrbot_description/urdf/rrbot_two.xacro (robot description, xacro)
@@ -48,7 +48,7 @@
     <parent link="link1"/>
     <child link="link2"/>
-    <origin xyz="0 ${width} ${height1 - axel_offset}" rpy="0 0 0"/>
+    <origin xyz="0 ${width} ${height1 - axel_offset}" rpy="0 ${-0.5*PI} 0"/>
     <axis xyz="0 1 0"/>
-    <limit effort="1000" lower="${-PI*2.0}" upper="${PI*2.0}" velocity="1"/>
+    <limit effort="10000" lower="${-PI*2.0}" upper="${PI*2.0}" velocity="1"/>
     <dynamics damping="0.1"/>
   </joint>
@@ -82,5 +82,5 @@
     <origin xyz="0 ${width} ${height2 - axel_offset*2}" rpy="0 0 0"/>
     <axis xyz="0 1 0"/>
-    <limit effort="1000" lower="${-PI*2.0}" upper="${PI*2.0}" velocity="1"/>
+    <limit effort="10000" lower="${-PI*2.0}" upper="${PI*2.0}" velocity="1"/>
     <dynamics damping="0.1"/>
   </joint>
@@ -162,7 +162,7 @@
     <parent link="link1_copy"/>
     <child link="link2_copy"/>
-    <origin xyz="0 ${width} ${height1 - axel_offset}" rpy="0 0 0"/>
+    <origin xyz="0 ${width} ${height1 - axel_offset}" rpy="0 ${0.5*PI} 0"/>
     <axis xyz="0 -1 0"/>
-    <limit effort="1000" lower="${-PI*2.0}" upper="${PI*2.0}" velocity="1"/>
+    <limit effort="10000" lower="${-PI*2.0}" upper="${PI*2.0}" velocity="1"/>
     <dynamics damping="0.1"/>
   </joint>
@@ -196,5 +196,5 @@
     <origin xyz="0 ${width} ${height2 - axel_offset*2}" rpy="0 0 0"/>
     <axis xyz="0 -1 0"/>
-    <limit effort="1000" lower="${-PI*2.0}" upper="${PI*2.0}" velocity="1"/>
+    <limit effort="10000" lower="${-PI*2.0}" upper="${PI*2.0}" velocity="1"/>
     <dynamics damping="0.1"/>
   </joint>
@@ -259,7 +259,4 @@
     <child link="box_copy"/>
     <origin xyz="0 ${width} ${height3 - axel_offset*2}" rpy="0 0 0"/>
-    <!-- <axis xyz="0 1 0"/> -->
-    <!-- <limit effort="1000" lower="${-PI*2.0}" upper="${PI*2.0}" velocity="1"/> -->
-    <!-- <dynamics damping="0.1"/> -->
   </joint>
   <transmission name="tran1_copy">
